Commit message: Revert "uploading data"
This reverts commit d581ebe8d526d545d1404a88b21d029682aafefe.

File: soft_hand_description/model/accesories/clamp.urdf.xacro (robot description, xacro)
@@ -1,27 +1,4 @@
 <?xml version="1.0"?>
 <robot xmlns:xacro="http://www.ros.org/wiki/xacro">
-<!--  Opened mesh /home/pacman/Projects/catkin_ws/src/vito-robot/pisa-iit-soft-hand/soft_hand_description/meshes/accesories/clamp.stl in 10 msec
-All files opened in 1273 msec
-Mesh Bounding Box Size 0,066000 0,072500 0,025600
-Mesh Bounding Box Diag 0,101329
-Mesh Volume is 0,000045
-Mesh Surface is 0,030645
-Thin shell barycenter -0,000000 -0,000183 -0,002245
-Center of Mass is -0,000000 -0,000206 -0,002440
-Inertia Tensor is :
-| 0,000000 -0,000000 0,000000 |
-| -0,000000 0,000000 -0,000000 |
-| 0,000000 -0,000000 0,000000 |
-Principal axes are :
-| 1,000000 0,000009 0,000002 |
-| -0,000009 1,000000 -0,000187 |
-| -0,000002 0,000187 1,000000 |
-axis momenta are :
-| 0,000000 0,000000 0,000000 |-->
-      <!-- conversions -->
-    <!-- I couldn't make the simulation work with realistic values, so I tweaked the conversion values -->
-    <xacro:property name="mm_to_m" value="0.001"/>
-    <xacro:property name="mm2_to_m2" value="0.000001"/>
-    <xacro:property name="gr_to_Kg" value="0.001"/>
 <xacro:macro name="clamp" params="parent name *origin">
   <joint name="${parent}_${name}_joint" type="fixed">
@@ -44,19 +21,5 @@
       </geometry>
     </collision>
-    <inertial>
-            <mass value="${150*gr_to_Kg}"/>
-        <inertia ixx="${150*gr_to_Kg * 66 * 66 * mm2_to_m2}" ixy="0.0" ixz="0.0" iyy="${150*gr_to_Kg * 72.5 * 72.5 * mm2_to_m2}" iyz="0.0" izz="${150*gr_to_Kg * 25.6*25.6 * mm2_to_m2}"/>
-      </inertial>
-	</link>
-      <gazebo reference="${name}">
-        <selfCollide>false</selfCollide>
-       <gravity>true</gravity>
-       <maxContacts>100</maxContacts>
-    <mu1>0.6</mu1>
-               <mu2>0.6</mu2>
-    <kp>1000000.0</kp>
-    <kd>1000.0</kd>
-    <minDepth>0.00</minDepth>
-   </gazebo>
+  </link>
 </xacro:macro>
 </robot>

File: soft_hand_description/model/accesories/kuka_coupler.urdf.xacro (robot description, xacro)
@@ -1,7 +1,4 @@
 <?xml version="1.0"?>
 <robot xmlns:xacro="http://www.ros.org/wiki/xacro">
-      <xacro:property name="mm_to_m" value="0.001"/>
-    <xacro:property name="mm2_to_m2" value="0.000001"/>
-    <xacro:property name="gr_to_Kg" value="0.001"/>
 <xacro:macro name="kuka_coupler" params="parent name *origin">
   <joint name="${parent}_${name}_joint" type="fixed">
@@ -25,9 +22,4 @@
       </geometry>
     </collision>
-        <inertial>
-      <origin xyz="0 0 0.031" rpy="0 0 0"/>
-        <mass value="${250*gr_to_Kg}"/>
-        <inertia ixx="${250*gr_to_Kg * 66 * 66 * mm2_to_m2}" ixy="0.0" ixz="0.0" iyy="${250*gr_to_Kg * 66* 66 * mm2_to_m2}" iyz="0.0" izz="${250*gr_to_Kg * 62 * 62 * mm2_to_m2}"/>
-      </inertial>
   </link>
   <joint name="${parent}_${name}_base_joint" type="fixed">
@@ -37,14 +29,4 @@
   </joint>
   <link name="${name}"/>
-      <gazebo reference="${name}_bottom">
-        <selfCollide>false</selfCollide>
-             <gravity>true</gravity>
-       <maxContacts>100</maxContacts>
-    <mu1>0.6</mu1>
-               <mu2>0.6</mu2>
-    <kp>1000000.0</kp>
-    <kd>1000.0</kd>
-    <minDepth>0.00</minDepth>
-   </gazebo>
 </xacro:macro>
 </robot>

File: soft_hand_description/model/accesories/softhand_base.urdf.xacro (robot description, xacro)
@@ -1,45 +1,4 @@
 <?xml version="1.0"?>
 <robot xmlns:xacro="http://www.ros.org/wiki/xacro">
-      <!-- conversions -->
-    <!-- I couldn't make the simulation work with realistic values, so I tweaked the conversion values -->
-    <xacro:property name="mm_to_m" value="0.001"/>
-    <xacro:property name="mm2_to_m2" value="0.000001"/>
-    <xacro:property name="gr_to_Kg" value="0.001"/>
-<!--Opened mesh /home/pacman/Projects/catkin_ws/src/vito-robot/pisa-iit-soft-hand/soft_hand_description/meshes/accesories/softhand_base_left.stl in 7 msec
-All files opened in 1341 msec
-Mesh Bounding Box Size 0,066000 0,066000 0,062000
-Mesh Bounding Box Diag 0,112054
-Mesh Volume is 0,000037
-Mesh Surface is 0,036962
-Thin shell barycenter -0,000349 0,000391 0,018653
-Center of Mass is -0,000229 0,000504 0,021471
-Inertia Tensor is :
-| 0,000000 0,000000 0,000000 |
-| 0,000000 0,000000 -0,000000 |
-| 0,000000 -0,000000 0,000000 |
-Principal axes are :
-| 0,989850 -0,140676 0,020182 |
-| 0,141292 0,989407 -0,033325 |
-| -0,015280 0,035838 0,999241 |
-axis momenta are :
-| 0,000000 0,000000 0,000000 |-->
-<!--Opened mesh /home/pacman/Projects/catkin_ws/src/vito-robot/pisa-iit-soft-hand/soft_hand_description/meshes/accesories/softhand_base_right.stl in 7 msec
-All files opened in 1390 msec
-Mesh Bounding Box Size 0,066000 0,066000 0,062000
-Mesh Bounding Box Diag 0,112054
-Mesh Volume is 0,000038
-Mesh Surface is 0,036673
-Thin shell barycenter -0,000377 -0,000489 0,019080
-Center of Mass is -0,000351 -0,000554 0,022132
-Inertia Tensor is :
-| 0,000000 -0,000000 0,000000 |
-| -0,000000 0,000000 0,000000 |
-| 0,000000 0,000000 0,000000 |
-Principal axes are :
-| 0,989801 0,140447 0,023852 |
-| -0,141290 0,989226 0,038338 |
-| -0,018210 -0,041317 0,998980 |
-axis momenta are :
-| 0,000000 0,000000 0,000000 |  -->
 <xacro:macro name="softhand_base" params="parent name left *origin">
   <joint name="${parent}_${name}_joint" type="fixed">
@@ -67,20 +26,5 @@
       </geometry>
     </collision>
-    <inertial>
-      <origin xyz="0 0 0.031" rpy="0 0 0"/>
-        <mass value="${250*gr_to_Kg}"/>
-        <inertia ixx="${250*gr_to_Kg * 66 * 66 * mm2_to_m2}" ixy="0.0" ixz="0.0" iyy="${250*gr_to_Kg * 66* 66 * mm2_to_m2}" iyz="0.0" izz="${250*gr_to_Kg * 62 * 62 * mm2_to_m2}"/>
-      </inertial>
   </link>
-    <gazebo reference="${name}">
-       <selfCollide>false</selfCollide>
-       <gravity>true</gravity>
-       <maxContacts>100</maxContacts>
-      <mu1>0.6</mu1>
-               <mu2>0.6</mu2>
-    <kp>1000000.0</kp>
-    <kd>1000.0</kd>
-    <minDepth>0.00</minDepth>
-   </gazebo>
 </xacro:macro>
 </robot>

File: soft_hand_description/model/soft_hand.gazebo.xacro (robot description, xacro)
@@ -620,31 +620,4 @@
 			<xacro:insert_block name="gazebo_joint_elements"/>
 		</gazebo>
-		  <gazebo>
-                     <plugin name="${name}_gazebo_gripper" filename="libvito_gazebo_gripper.so">
-		    <updateRate>1000.0</updateRate>
-		       <gripperAttachLink>${name}_thumb_knuckle_link</gripperAttachLink>
- 		       <gripperLink>${name}_thumb_distal_link</gripperLink>
-		       <gripperLink>${name}_thumb_proximal_link</gripperLink>
-		        <gripperLink>${name}_index_knuckle_link</gripperLink>
-			<gripperLink>${name}_index_proximal_link</gripperLink>
-			<gripperLink>${name}_index_middle_link</gripperLink>
- 			<gripperLink>${name}_index_distal_link</gripperLink>
-			<gripperLink>${name}_middle_knuckle_link</gripperLink>
-			<gripperLink>${name}_middle_proximal_link</gripperLink>
-                       <gripperLink>${name}_middle_middle_link</gripperLink>
- 			<gripperLink>${name}_middle_distal_link</gripperLink>
-			<gripperLink>${name}_ring_knuckle_link</gripperLink>
-			<gripperLink>${name}_ring_proximal_link</gripperLink>
-			<gripperLink>${name}_ring_middle_link</gripperLink>
-                        <gripperLink>${name}_ring_distal_link</gripperLink>
-			<gripperLink>${name}_little_knuckle_link</gripperLink>
-			<gripperLink>${name}_little_proximal_link</gripperLink>
-                       <gripperLink>${name}_little_middle_link</gripperLink>
- 			<gripperLink>${name}_little_distal_link</gripperLink>
-                       <maxRelativeMotionRate>0.001</maxRelativeMotionRate>
-                       <attachWait>0.1</attachWait>
-                       <detachWait>0.0</detachWait>
-                   </plugin>
-		 </gazebo>
 	</xacro:macro>
 </robot>

File: soft_hand_description/model/soft_hand.inertia.xacro (robot description, xacro)
@@ -9,6 +9,6 @@
     <!-- I couldn't make the simulation work with realistic values, so I tweaked the conversion values -->
     <xacro:property name="mm_to_m" value="0.001"/>
-     <xacro:property name="mm2_to_m2" value="0.000001"/>
-    <xacro:property name="gr_to_Kg" value="0.001"/>
+    <xacro:property name="mm2_to_m2" value="0.001"/>
+    <xacro:property name="gr_to_Kg" value="0.01"/>
     <!-- not so negligible, otherwise simulation fails -->
     <xacro:property name="negligible_mass" value="${10*gr_to_Kg}"/>
@@ -131,5 +131,5 @@
 Mesh Volume is 76748.765625
 Mesh Surface is 52111.375000
-Thin shell barycenter -5.584415 -7.926011 28.832655aaaaaaaaaaaaaaaaaaaaaa
+Thin shell barycenter -5.584415 -7.926011 28.832655
 Center of Mass is -4.568758 -6.808116 27.653328
 Inertia Tensor is :
