Commit message: Revert "uploading data"
This reverts commit d581ebe8d526d545d1404a88b21d029682aafefe.

File: soft_hand_description/model/soft_hand.transmission.xacro (robot description, xacro)
@@ -131,18 +131,17 @@
     </xacro:unless>
     <xacro:if value="${withAdaptiveTransmission}">
-   <!-- work in progress -->
-   <transmission name="${name}_synergy_trans">
-       <robotNamespace>${name}</robotNamespace>
-       <type>transmission_interface/SimpleTransmission</type>
-       <joint name="${name}_synergy_joint">
-          <hardwareInterface>PositionJointInterface</hardwareInterface>
-	<!-- <hardwareInterface>EffortJointInterface</hardwareInterface>-->
-       </joint>
-       <actuator name="${name}_synergy_motor">
-         <mechanicalReduction>1.0</mechanicalReduction>
-<!-- 	  <mechanicalElasticity>1.0</mechanicalElasticity> -->
-       </actuator>
-   </transmission>
-    <transmission name="${name}_joint_trans">
+      <!-- work in progress -->
+      <transmission name="${name}_synergy_trans">
+          <robotNamespace>${name}</robotNamespace>
+          <type>transmission_interface/SimpleTransmission</type>
+          <joint name="${name}_synergy_joint">
+            <hardwareInterface>PositionJointInterface</hardwareInterface>
+            <!--hardwareInterface>EffortJointInterface</hardwareInterface-->
+          </joint>
+          <actuator name="${name}_synergy_motor">
+            <mechanicalReduction>1.0</mechanicalReduction>
+          </actuator>
+      </transmission>
+      <transmission name="${name}_joint_trans">
         <robotNamespace>${name}</robotNamespace>
         <type>transmission_interface/AdaptiveSynergyTransmission</type>
@@ -151,8 +150,7 @@
             <offset>-0.0</offset>
             <mechanicalReduction>1.3</mechanicalReduction>
-           <!-- <mechanicalElasticity>0.001</mechanicalElasticity>-->
-             <mechanicalElasticity>1.0</mechanicalElasticity>
-	    <hardwareInterface>PositionJointInterface</hardwareInterface>
-<!--             <hardwareInterface>EffortJointInterface</hardwareInterface> -->
+            <mechanicalElasticity>1.0</mechanicalElasticity>
+            <!-- hardwareInterface>PositionJointInterface</hardwareInterface -->
+            <hardwareInterface>EffortJointInterface</hardwareInterface>
           </joint>
           <joint name="${name}_thumb_inner_joint">
@@ -160,7 +158,7 @@
             <offset>-0.0</offset>
             <mechanicalReduction>1.0</mechanicalReduction>
-            <mechanicalElasticity>0.001</mechanicalElasticity>
-	    <hardwareInterface>PositionJointInterface</hardwareInterface>
-<!--             <hardwareInterface>EffortJointInterface</hardwareInterface> -->
+            <mechanicalElasticity>1.0</mechanicalElasticity>
+            <!-- hardwareInterface>PositionJointInterface</hardwareInterface -->
+            <hardwareInterface>EffortJointInterface</hardwareInterface>
           </joint>
           <joint name="${name}_thumb_outer_joint">
@@ -168,149 +166,146 @@
             <offset>-0.0</offset>
             <mechanicalReduction>1.0</mechanicalReduction>
-            <mechanicalElasticity>0.001</mechanicalElasticity>
-            <hardwareInterface>PositionJointInterface</hardwareInterface>
-<!--             <hardwareInterface>EffortJointInterface</hardwareInterface> -->
-          </joint>
-       <joint name="${name}_index_abd_joint">
-         <role>joint4</role>
-         <offset>-0.0</offset>
-	 <mechanicalReduction>0.5</mechanicalReduction>
-         <mechanicalElasticity>2.0</mechanicalElasticity>
-        <hardwareInterface>PositionJointInterface</hardwareInterface>
-         <!--<hardwareInterface>EffortJointInterface</hardwareInterface>-->
-       </joint>
-       <joint name="${name}_index_inner_joint">
-         <role>joint5</role>
-         <offset>-0.0</offset>
-         <mechanicalReduction>1.0</mechanicalReduction>
-         <mechanicalElasticity>1.0</mechanicalElasticity>
-         <hardwareInterface>PositionJointInterface</hardwareInterface>
-         <!--<hardwareInterface>EffortJointInterface</hardwareInterface>-->
-       </joint>
-       <joint name="${name}_index_middle_joint">
-         <role>joint6</role>
-         <offset>-0.0</offset>
-         <mechanicalReduction>1.0</mechanicalReduction>
-         <mechanicalElasticity>1.0</mechanicalElasticity>
-         <hardwareInterface>PositionJointInterface</hardwareInterface>
-         <!--<hardwareInterface>EffortJointInterface</hardwareInterface>-->
-       </joint>
-       <joint name="${name}_index_outer_joint">
-         <role>joint7</role>
-         <offset>-0.0</offset>
-         <mechanicalReduction>1.0</mechanicalReduction>
-         <mechanicalElasticity>1.0</mechanicalElasticity>
-        <hardwareInterface>PositionJointInterface</hardwareInterface>
-         <!--<hardwareInterface>EffortJointInterface</hardwareInterface>-->
-       </joint>
-       <joint name="${name}_middle_abd_joint">
-         <role>joint8</role>
-         <offset>-0.0</offset>
-          <mechanicalReduction>0.5</mechanicalReduction>
-         <mechanicalElasticity>1.0</mechanicalElasticity>
-         <hardwareInterface>PositionJointInterface</hardwareInterface>
-         <!--<hardwareInterface>EffortJointInterface</hardwareInterface>-->
-       </joint>
-       <joint name="${name}_middle_inner_joint">
-         <role>joint9</role>
-         <offset>-0.0</offset>
-         <mechanicalReduction>1.0</mechanicalReduction>
-         <mechanicalElasticity>1.0</mechanicalElasticity>
-        <hardwareInterface>PositionJointInterface</hardwareInterface>
-         <!--<hardwareInterface>EffortJointInterface</hardwareInterface>-->
-       </joint>
-       <joint name="${name}_middle_middle_joint">
-         <role>joint10</role>
-         <offset>-0.0</offset>
-         <mechanicalReduction>1.0</mechanicalReduction>
-         <mechanicalElasticity>1.0</mechanicalElasticity>
-        <hardwareInterface>PositionJointInterface</hardwareInterface>
-         <!--<hardwareInterface>EffortJointInterface</hardwareInterface>-->
-       </joint>
-       <joint name="${name}_middle_outer_joint">
-         <role>joint11</role>
-         <offset>-0.0</offset>
-         <mechanicalReduction>1.0</mechanicalReduction>
-         <mechanicalElasticity>1.0</mechanicalElasticity>
-        <hardwareInterface>PositionJointInterface</hardwareInterface>
-         <!--<hardwareInterface>EffortJointInterface</hardwareInterface>-->
-       </joint>
-       <joint name="${name}_ring_abd_joint">
-         <role>joint12</role>
-         <offset>-0.0</offset>
-<!-- 	 <mechanicalReduction>0.2</mechanicalReduction> -->
-         <mechanicalReduction>0.5</mechanicalReduction>
-	 <mechanicalElasticity>1.0</mechanicalElasticity>
-         <hardwareInterface>PositionJointInterface</hardwareInterface>
-       <!--  <hardwareInterface>EffortJointInterface</hardwareInterface>-->
-       </joint>
-       <joint name="${name}_ring_inner_joint">
-         <role>joint13</role>
-         <offset>-0.0</offset>
-         <mechanicalReduction>1.0</mechanicalReduction>
-         <mechanicalElasticity>1.0</mechanicalElasticity>
-         <hardwareInterface>PositionJointInterface</hardwareInterface>
-         <!--<hardwareInterface>EffortJointInterface</hardwareInterface>-->
-       </joint>
-       <joint name="${name}_ring_middle_joint">
-         <role>joint14</role>
-         <offset>-0.0</offset>
-         <mechanicalReduction>1.0</mechanicalReduction>
-         <mechanicalElasticity>1.0</mechanicalElasticity>
-        <hardwareInterface>PositionJointInterface</hardwareInterface>
-         <!--<hardwareInterface>EffortJointInterface</hardwareInterface>-->
-       </joint>
-       <joint name="${name}_ring_outer_joint">
-         <role>joint15</role>
-         <offset>-0.0</offset>
-         <mechanicalReduction>1.0</mechanicalReduction>
-         <mechanicalElasticity>1.0</mechanicalElasticity>
-         <hardwareInterface>PositionJointInterface</hardwareInterface>
-         <!--<hardwareInterface>EffortJointInterface</hardwareInterface>-->
-       </joint>
-       <joint name="${name}_little_abd_joint">
-         <role>joint16</role>
-         <offset>-0.0</offset>
-<!--           <mechanicalReduction>0.4</mechanicalReduction> -->
-         <mechanicalReduction>0.5</mechanicalReduction>
-	 <mechanicalElasticity>1.0</mechanicalElasticity>
-         <hardwareInterface>PositionJointInterface</hardwareInterface>
-<!--          <hardwareInterface>EffortJointInterface</hardwareInterface> -->
-       </joint>
-       <joint name="${name}_little_inner_joint">
-         <role>joint17</role>
-         <offset>-0.0</offset>
-         <mechanicalReduction>1.0</mechanicalReduction>
-         <mechanicalElasticity>1.0</mechanicalElasticity>
-         <hardwareInterface>PositionJointInterface</hardwareInterface>
-<!--          <hardwareInterface>EffortJointInterface</hardwareInterface> -->
-       </joint>
-       <joint name="${name}_little_middle_joint">
-         <role>joint18</role>
-         <offset>-0.0</offset>
-         <mechanicalReduction>1.0</mechanicalReduction>
-         <mechanicalElasticity>1.0</mechanicalElasticity>
-         <hardwareInterface>PositionJointInterface</hardwareInterface>
-<!--          <hardwareInterface>EffortJointInterface</hardwareInterface> -->
-       </joint>
-       <joint name="${name}_little_outer_joint">
-         <role>joint19</role>
-         <offset>-0.0</offset>
-         <mechanicalReduction>1.0</mechanicalReduction>
-         <mechanicalElasticity>1.0</mechanicalElasticity>
-         <hardwareInterface>PositionJointInterface</hardwareInterface>
-<!--          <hardwareInterface>EffortJointInterface</hardwareInterface> -->
-       </joint>
-       <!-- IMPORTANT: if you change the elasticity or reduction at the joints, this value must be calibrated again to
-                       ensure that the joints don't go after the limits -->
-       <!-- ToDO: autocalibration using the joint limits. When the synergy goes to 1, they must be at the upper limirt
-                 and to 0, they must be at the lower limit -->
-       <actuator name="${name}_actuator">
-         <role>actuator1</role>
-         <mechanicalReduction>4.5</mechanicalReduction>
-	  <!--<mechanicalElasticity>5.0</mechanicalElasticity>-->
-       </actuator>
-   </transmission>
- </xacro:if>
+            <mechanicalElasticity>1.0</mechanicalElasticity>
+            <!-- hardwareInterface>PositionJointInterface</hardwareInterface -->
+            <hardwareInterface>EffortJointInterface</hardwareInterface>
+          </joint>
+          <joint name="${name}_index_abd_joint">
+            <role>joint4</role>
+            <offset>-0.0</offset>
+            <mechanicalReduction>-0.2</mechanicalReduction>
+            <mechanicalElasticity>1.0</mechanicalElasticity>
+            <!-- hardwareInterface>PositionJointInterface</hardwareInterface -->
+            <hardwareInterface>EffortJointInterface</hardwareInterface>
+          </joint>
+          <joint name="${name}_index_inner_joint">
+            <role>joint5</role>
+            <offset>-0.0</offset>
+            <mechanicalReduction>1.0</mechanicalReduction>
+            <mechanicalElasticity>1.0</mechanicalElasticity>
+            <!-- hardwareInterface>PositionJointInterface</hardwareInterface -->
+            <hardwareInterface>EffortJointInterface</hardwareInterface>
+          </joint>
+          <joint name="${name}_index_middle_joint">
+            <role>joint6</role>
+            <offset>-0.0</offset>
+            <mechanicalReduction>1.0</mechanicalReduction>
+            <mechanicalElasticity>1.0</mechanicalElasticity>
+            <!-- hardwareInterface>PositionJointInterface</hardwareInterface -->
+            <hardwareInterface>EffortJointInterface</hardwareInterface>
+          </joint>
+          <joint name="${name}_index_outer_joint">
+            <role>joint7</role>
+            <offset>-0.0</offset>
+            <mechanicalReduction>1.0</mechanicalReduction>
+            <mechanicalElasticity>1.0</mechanicalElasticity>
+            <!-- hardwareInterface>PositionJointInterface</hardwareInterface -->
+            <hardwareInterface>EffortJointInterface</hardwareInterface>
+          </joint>
+          <joint name="${name}_middle_abd_joint">
+            <role>joint8</role>
+            <offset>-0.0</offset>
+            <mechanicalReduction>0.001</mechanicalReduction>
+            <mechanicalElasticity>1.0</mechanicalElasticity>
+            <!-- hardwareInterface>PositionJointInterface</hardwareInterface -->
+            <hardwareInterface>EffortJointInterface</hardwareInterface>
+          </joint>
+          <joint name="${name}_middle_inner_joint">
+            <role>joint9</role>
+            <offset>-0.0</offset>
+            <mechanicalReduction>1.0</mechanicalReduction>
+            <mechanicalElasticity>1.0</mechanicalElasticity>
+            <!-- hardwareInterface>PositionJointInterface</hardwareInterface -->
+            <hardwareInterface>EffortJointInterface</hardwareInterface>
+          </joint>
+          <joint name="${name}_middle_middle_joint">
+            <role>joint10</role>
+            <offset>-0.0</offset>
+            <mechanicalReduction>1.0</mechanicalReduction>
+            <mechanicalElasticity>1.0</mechanicalElasticity>
+            <!-- hardwareInterface>PositionJointInterface</hardwareInterface -->
+            <hardwareInterface>EffortJointInterface</hardwareInterface>
+          </joint>
+          <joint name="${name}_middle_outer_joint">
+            <role>joint11</role>
+            <offset>-0.0</offset>
+            <mechanicalReduction>1.0</mechanicalReduction>
+            <mechanicalElasticity>1.0</mechanicalElasticity>
+            <!-- hardwareInterface>PositionJointInterface</hardwareInterface -->
+            <hardwareInterface>EffortJointInterface</hardwareInterface>
+          </joint>
+          <joint name="${name}_ring_abd_joint">
+            <role>joint12</role>
+            <offset>-0.0</offset>
+            <mechanicalReduction>0.2</mechanicalReduction>
+            <mechanicalElasticity>1.0</mechanicalElasticity>
+            <!-- hardwareInterface>PositionJointInterface</hardwareInterface -->
+            <hardwareInterface>EffortJointInterface</hardwareInterface>
+          </joint>
+          <joint name="${name}_ring_inner_joint">
+            <role>joint13</role>
+            <offset>-0.0</offset>
+            <mechanicalReduction>1.0</mechanicalReduction>
+            <mechanicalElasticity>1.0</mechanicalElasticity>
+            <!-- hardwareInterface>PositionJointInterface</hardwareInterface -->
+            <hardwareInterface>EffortJointInterface</hardwareInterface>
+          </joint>
+          <joint name="${name}_ring_middle_joint">
+            <role>joint14</role>
+            <offset>-0.0</offset>
+            <mechanicalReduction>1.0</mechanicalReduction>
+            <mechanicalElasticity>1.0</mechanicalElasticity>
+            <!-- hardwareInterface>PositionJointInterface</hardwareInterface -->
+            <hardwareInterface>EffortJointInterface</hardwareInterface>
+          </joint>
+          <joint name="${name}_ring_outer_joint">
+            <role>joint15</role>
+            <offset>-0.0</offset>
+            <mechanicalReduction>1.0</mechanicalReduction>
+            <mechanicalElasticity>1.0</mechanicalElasticity>
+            <!-- hardwareInterface>PositionJointInterface</hardwareInterface -->
+            <hardwareInterface>EffortJointInterface</hardwareInterface>
+          </joint>
+          <joint name="${name}_little_abd_joint">
+            <role>joint16</role>
+            <offset>-0.0</offset>
+            <mechanicalReduction>0.4</mechanicalReduction>
+            <mechanicalElasticity>1.0</mechanicalElasticity>
+            <!-- hardwareInterface>PositionJointInterface</hardwareInterface -->
+            <hardwareInterface>EffortJointInterface</hardwareInterface>
+          </joint>
+          <joint name="${name}_little_inner_joint">
+            <role>joint17</role>
+            <offset>-0.0</offset>
+            <mechanicalReduction>1.0</mechanicalReduction>
+            <mechanicalElasticity>1.0</mechanicalElasticity>
+            <!-- hardwareInterface>PositionJointInterface</hardwareInterface -->
+            <hardwareInterface>EffortJointInterface</hardwareInterface>
+          </joint>
+          <joint name="${name}_little_middle_joint">
+            <role>joint18</role>
+            <offset>-0.0</offset>
+            <mechanicalReduction>1.0</mechanicalReduction>
+            <mechanicalElasticity>1.0</mechanicalElasticity>
+            <!-- hardwareInterface>PositionJointInterface</hardwareInterface -->
+            <hardwareInterface>EffortJointInterface</hardwareInterface>
+          </joint>
+          <joint name="${name}_little_outer_joint">
+            <role>joint19</role>
+            <offset>-0.0</offset>
+            <mechanicalReduction>1.0</mechanicalReduction>
+            <mechanicalElasticity>1.0</mechanicalElasticity>
+            <!-- hardwareInterface>PositionJointInterface</hardwareInterface -->
+            <hardwareInterface>EffortJointInterface</hardwareInterface>
+          </joint>
+          <!-- IMPORTANT: if you change the elasticity or reduction at the joints, this value must be calibrated again to
+                          ensure that the joints don't go after the limits -->
+          <!-- ToDO: autocalibration using the joint limits. When the synergy goes to 1, they must be at the upper limirt
+                    and to 0, they must be at the lower limit -->
+          <actuator name="${name}_actuator">
+            <role>actuator1</role>
+            <mechanicalReduction>4.5</mechanicalReduction>
+          </actuator>
+      </transmission>
+    </xacro:if>
   </xacro:macro>
 </robot>

File: soft_hand_description/model/soft_hand.urdf.xacro (robot description, xacro)
@@ -14,5 +14,5 @@
 	<xacro:property name="abd_lb" value="-30" />
 	<xacro:property name="abd_ub" value="30" />
-	<xacro:property name="thumb_abd_lb" value="0" />  <!-- 75 -->
+	<xacro:property name="thumb_abd_lb" value="0" />
 	<xacro:property name="thumb_abd_ub" value="90" />
 	<xacro:property name="inner_lb" value="0" />
@@ -21,20 +21,14 @@
 	<xacro:property name="middle_ub" value="45" />
 	<xacro:property name="outer_lb" value="0" />
-	<xacro:property name="outer_ub" value="35" />
+	<xacro:property name="outer_ub" value="45" />
 	<xacro:property name="velocity" value="100" />
 	<xacro:property name="effort" value="100" />
-	<xacro:property name="damping" value="100" />
-	<xacro:property name="friction" value="10.0" />
-<!-- 	<xacro:property name="inner_lb" value="0" />
-	<xacro:property name="inner_ub" value="5" />
-	<xacro:property name="middle_lb" value="0" />
-	<xacro:property name="middle_ub" value="5" />
-	<xacro:property name="outer_lb" value="0" />
-	<xacro:property name="outer_ub" value="5" /> -->
+	<xacro:property name="damping" value="0.0" />
+	<xacro:property name="friction" value="0.0" />
 	<!-- synergy vector -->
 	<xacro:property name="syn_amp" value="1" />
 	<xacro:property name="thumb_abd_R" value="${1.3*syn_amp}" />
 	<xacro:property name="thumb_inner_R" value="${1.3*syn_amp}" />
-	<xacro:property name="thumb_outer_R" value="${1.3*syn_amp}" />
+	<xacro:property name="thumb_outer_R" value="${1.0*syn_amp}" />
 	<xacro:property name="index_abd_R" value="-${0.2*syn_amp}" />
 	<xacro:property name="index_inner_R" value="${1.0*syn_amp}" />
@@ -58,6 +52,6 @@
 	<xacro:property name="max_synergy_velocity" value="100000" />
 	<xacro:property name="max_synergy_effort" value="100" />
-	<xacro:property name="synergy_damping" value="2.0" />
-	<xacro:property name="synergy_friction" value="2.0" />
+	<xacro:property name="synergy_damping" value="0.0" />
+	<xacro:property name="synergy_friction" value="0.0" />
 	<!-- SOFT FINGER model -->
 	<!-- 4 fingers are equal (index, middle, ring, little) -->
@@ -243,5 +237,4 @@
 				<xacro:if value="${useMimicTag}">
 					<mimic joint="${parent_name}_synergy_joint" multiplier="${abd_R}"/>
-					<!-- <mimic joint="${parent_name}_synergy_joint" multiplier="${abd_R}"/> -->
 				</xacro:if>
 			</joint>
@@ -452,23 +445,4 @@
 			</xacro:unless>
 		</link>
-<!--
-		 PALM  dummy
- 		<joint name="${name}_palm_joint_dummy" type="revolute">
-			<xacro:if value="${left}">
-				<origin xyz="0.00 0.0 0.10" rpy="0 0 0"/>
-				<limit lower="0" upper="0" effort="0" velocity="0"/>
-			</xacro:if>
-			<xacro:unless value="${left}">
-				<origin xyz="0.00 +0.0 0.10" rpy="0 0 0"/>
- 				<limit lower="0" upper="0" effort="0" velocity="0"/>
-			</xacro:unless>
-			<parent link="${name}_palm_link" />
-			<child link="${name}_palm_dummy_link" />
-		</joint>
-		<link name="${name}_palm_dummy_link">
-			<inertial>
-				<insert_block name="negligible_inertia"/>
-			</inertial>
-		</link> -->
 		<!-- MOTOR JOINT -->
 		<joint name="${name}_synergy_joint" type="revolute" >
@@ -495,5 +469,4 @@
 		<xacro:unless value="${left}">
 			<xacro:soft_thumb parent="${name}_palm_link" parent_name="${name}" name="${name}_thumb" position="0.00566972 0.0296160 0.0553140" orientation="0.0 -0.38397275793662144 1.5707963267948966" left="${left}" useMimicTag="${useMimicTag}" abd_R="${thumb_abd_R *(thumb_abd_ub - thumb_abd_lb)*pi/180}" inner_R="${thumb_inner_R *(inner_ub - inner_lb)*pi/180}" outer_R="${thumb_outer_R *(outer_ub - outer_lb)*pi/180}"/>
-<!-- <xacro:soft_thumb parent="${name}_palm_link" parent_name="${name}" name="${name}_thumb" position="0.00966972 0.0396160 0.0653140" orientation="0.0 -0.38397275793662144 1.5707963267948966" left="${left}" useMimicTag="${useMimicTag}" abd_R="${thumb_abd_R *(thumb_abd_ub - thumb_abd_lb)*pi/180}" inner_R="${thumb_inner_R *(inner_ub - inner_lb)*pi/180}" outer_R="${thumb_outer_R *(outer_ub - outer_lb)*pi/180}"/>-->
 			<xacro:soft_finger parent="${name}_palm_link" parent_name="${name}" name="${name}_index" position="-0.0033 0.0195 0.0936994" orientation="1.5707963267948966 -1.4835299330931884 1.5707963267948966" left="${left}" useMimicTag="${useMimicTag}" abd_R="${index_abd_R}" inner_R="${index_inner_R *(inner_ub - inner_lb)*pi/180}" middle_R="${index_middle_R *(middle_ub - middle_lb)*pi/180}" outer_R="${index_outer_R *(outer_ub - outer_lb)*pi/180}" />
 			<xacro:soft_finger parent="${name}_palm_link" parent_name="${name}" name="${name}_middle" position="-0.003300000 0.0 0.100699" orientation="3.141592 -1.5707963267948966 0.0" left="${left}" useMimicTag="${useMimicTag}" abd_R="${middle_abd_R}" inner_R="${middle_inner_R *(inner_ub - inner_lb)*pi/180}" middle_R="${middle_middle_R *(middle_ub - middle_lb)*pi/180}" outer_R="${middle_outer_R *(outer_ub - outer_lb)*pi/180}" />
