Commit message: sensor fusion hand

File: soft_hand_description/model/soft_hand.gazebo.xacro (robot description, xacro)
@@ -58,8 +58,10 @@
 			<!--selfCollide>true</selfCollide-->
 			<gravity>true</gravity>
-			<mu1>500.0</mu1>
-			<mu2>500.0</mu2>
-			<kp>10000000.0</kp>
-			<kd>1.0</kd>
+			<mu1>1.0</mu1>
+			<mu2>1.0</mu2>
+			<kp>500000.0</kp>
+			<kd>1000.0</kd>
+			<minDepth>0.00</minDepth>
+			<maxVel>0.00</maxVel>
 		</gazebo>
 		<gazebo reference="${name}_thumb_knuckle_link">
@@ -82,8 +84,10 @@
 			<!--selfCollide>true</selfCollide-->
 			<gravity>true</gravity>
-			<mu1>500.0</mu1>
-			<mu2>500.0</mu2>
-			<kp>10000000.0</kp>
-			<kd>1.0</kd>
+			<mu1>1.0</mu1>
+			<mu2>1.0</mu2>
+			<kp>500000.0</kp>
+			<kd>1000.0</kd>
+			<minDepth>0.00</minDepth>
+			<maxVel>0.00</maxVel>
 		</gazebo>
 		<gazebo reference="${name}_thumb_proximal_link">
@@ -106,8 +110,10 @@
 			<!--selfCollide>true</selfCollide-->
 			<gravity>true</gravity>
-			<mu1>500.0</mu1>
-			<mu2>500.0</mu2>
-			<kp>10000000.0</kp>
-			<kd>1.0</kd>
+			<mu1>1.0</mu1>
+			<mu2>1.0</mu2>
+			<kp>500000.0</kp>
+			<kd>1000.0</kd>
+			<minDepth>0.00</minDepth>
+			<maxVel>0.00</maxVel>
 		</gazebo>
 		<gazebo reference="${name}_thumb_distal_link">
@@ -130,8 +136,10 @@
 			<!-- selfCollide>true</selfCollide-->
 			<gravity>true</gravity>
-			<mu1>500.0</mu1>
-			<mu2>500.0</mu2>
-			<kp>10000000.0</kp>
-			<kd>1.0</kd>
+			<mu1>1.0</mu1>
+			<mu2>1.0</mu2>
+			<kp>500000.0</kp>
+			<kd>1000.0</kd>
+			<minDepth>0.00</minDepth>
+			<maxVel>0.00</maxVel>
 		</gazebo>
 		<gazebo reference="${name}_index_knuckle_link">
@@ -154,8 +162,10 @@
 			<!--selfCollide>true</selfCollide-->
 			<gravity>true</gravity>
-			<mu1>500.0</mu1>
-			<mu2>500.0</mu2>
-			<kp>10000000.0</kp>
-			<kd>1.0</kd>
+			<mu1>1.0</mu1>
+			<mu2>1.0</mu2>
+			<kp>500000.0</kp>
+			<kd>1000.0</kd>
+			<minDepth>0.00</minDepth>
+			<maxVel>0.00</maxVel>
 		</gazebo>
 		<gazebo reference="${name}_index_proximal_link">
@@ -178,8 +188,10 @@
 			<!--selfCollide>true</selfCollide-->
 			<gravity>true</gravity>
-			<mu1>500.0</mu1>
-			<mu2>500.0</mu2>
-			<kp>10000000.0</kp>
-			<kd>1.0</kd>
+			<mu1>1.0</mu1>
+			<mu2>1.0</mu2>
+			<kp>500000.0</kp>
+			<kd>1000.0</kd>
+			<minDepth>0.00</minDepth>
+			<maxVel>0.00</maxVel>
 		</gazebo>
 		<gazebo reference="${name}_index_middle_link">
@@ -202,8 +214,10 @@
 			<!--selfCollide>true</selfCollide-->
 			<gravity>true</gravity>
-			<mu1>500.0</mu1>
-			<mu2>500.0</mu2>
-			<kp>10000000.0</kp>
-			<kd>1.0</kd>
+			<mu1>1.0</mu1>
+			<mu2>1.0</mu2>
+			<kp>500000.0</kp>
+			<kd>1000.0</kd>
+			<minDepth>0.00</minDepth>
+			<maxVel>0.00</maxVel>
 		</gazebo>
 		<gazebo reference="${name}_index_distal_link">
@@ -226,8 +240,10 @@
 			<!-- selfCollide>true</selfCollide-->
 			<gravity>true</gravity>
-			<mu1>500.0</mu1>
-			<mu2>500.0</mu2>
-			<kp>10000000.0</kp>
-			<kd>1.0</kd>
+			<mu1>1.0</mu1>
+			<mu2>1.0</mu2>
+			<kp>500000.0</kp>
+			<kd>1000.0</kd>
+			<minDepth>0.00</minDepth>
+			<maxVel>0.00</maxVel>
 		</gazebo>
 		<gazebo reference="${name}_middle_knuckle_link">
@@ -250,8 +266,10 @@
 			<!--selfCollide>true</selfCollide-->
 			<gravity>true</gravity>
-			<mu1>500.0</mu1>
-			<mu2>500.0</mu2>
-			<kp>10000000.0</kp>
-			<kd>1.0</kd>
+			<mu1>1.0</mu1>
+			<mu2>1.0</mu2>
+			<kp>500000.0</kp>
+			<kd>1000.0</kd>
+			<minDepth>0.00</minDepth>
+			<maxVel>0.00</maxVel>
 		</gazebo>
 		<gazebo reference="${name}_middle_proximal_link">
@@ -274,8 +292,10 @@
 			<!--selfCollide>true</selfCollide-->
 			<gravity>true</gravity>
-			<mu1>500.0</mu1>
-			<mu2>500.0</mu2>
-			<kp>10000000.0</kp>
-			<kd>1.0</kd>
+			<mu1>1.0</mu1>
+			<mu2>1.0</mu2>
+			<kp>500000.0</kp>
+			<kd>1000.0</kd>
+			<minDepth>0.00</minDepth>
+			<maxVel>0.00</maxVel>
 		</gazebo>
 		<gazebo reference="${name}_middle_middle_link">
@@ -298,8 +318,10 @@
 			<!--selfCollide>true</selfCollide-->
 			<gravity>true</gravity>
-			<mu1>500.0</mu1>
-			<mu2>500.0</mu2>
-			<kp>10000000.0</kp>
-			<kd>1.0</kd>
+			<mu1>1.0</mu1>
+			<mu2>1.0</mu2>
+			<kp>500000.0</kp>
+			<kd>1000.0</kd>
+			<minDepth>0.00</minDepth>
+			<maxVel>0.00</maxVel>
 		</gazebo>
 		<gazebo reference="${name}_middle_distal_link">
@@ -322,8 +344,10 @@
 			<!-- selfCollide>true</selfCollide-->
 			<gravity>true</gravity>
-			<mu1>500.0</mu1>
-			<mu2>500.0</mu2>
-			<kp>10000000.0</kp>
-			<kd>1.0</kd>
+			<mu1>1.0</mu1>
+			<mu2>1.0</mu2>
+			<kp>500000.0</kp>
+			<kd>1000.0</kd>
+			<minDepth>0.00</minDepth>
+			<maxVel>0.00</maxVel>
 		</gazebo>
 		<gazebo reference="${name}_ring_knuckle_link">
@@ -346,8 +370,10 @@
 			<!--selfCollide>true</selfCollide-->
 			<gravity>true</gravity>
-			<mu1>500.0</mu1>
-			<mu2>500.0</mu2>
-			<kp>10000000.0</kp>
-			<kd>1.0</kd>
+			<mu1>1.0</mu1>
+			<mu2>1.0</mu2>
+			<kp>500000.0</kp>
+			<kd>1000.0</kd>
+			<minDepth>0.00</minDepth>
+			<maxVel>0.00</maxVel>
 		</gazebo>
 		<gazebo reference="${name}_ring_proximal_link">
@@ -370,8 +396,10 @@
 			<!--selfCollide>true</selfCollide-->
 			<gravity>true</gravity>
-			<mu1>500.0</mu1>
-			<mu2>500.0</mu2>
-			<kp>10000000.0</kp>
-			<kd>1.0</kd>
+			<mu1>1.0</mu1>
+			<mu2>1.0</mu2>
+			<kp>500000.0</kp>
+			<kd>1000.0</kd>
+			<minDepth>0.00</minDepth>
+			<maxVel>0.00</maxVel>
 		</gazebo>
 		<gazebo reference="${name}_ring_middle_link">
@@ -394,8 +422,10 @@
 			<!--selfCollide>true</selfCollide-->
 			<gravity>true</gravity>
-			<mu1>500.0</mu1>
-			<mu2>500.0</mu2>
-			<kp>10000000.0</kp>
-			<kd>1.0</kd>
+			<mu1>1.0</mu1>
+			<mu2>1.0</mu2>
+			<kp>500000.0</kp>
+			<kd>1000.0</kd>
+			<minDepth>0.00</minDepth>
+			<maxVel>0.00</maxVel>
 		</gazebo>
 		<gazebo reference="${name}_ring_distal_link">
@@ -418,8 +448,10 @@
 			<!-- selfCollide>true</selfCollide-->
 			<gravity>true</gravity>
-			<mu1>500.0</mu1>
-			<mu2>500.0</mu2>
-			<kp>10000000.0</kp>
-			<kd>1.0</kd>
+			<mu1>1.0</mu1>
+			<mu2>1.0</mu2>
+			<kp>500000.0</kp>
+			<kd>1000.0</kd>
+			<minDepth>0.00</minDepth>
+			<maxVel>0.00</maxVel>
 		</gazebo>
 		<gazebo reference="${name}_little_knuckle_link">
@@ -442,8 +474,10 @@
 			<!--selfCollide>true</selfCollide-->
 			<gravity>true</gravity>
-			<mu1>500.0</mu1>
-			<mu2>500.0</mu2>
-			<kp>10000000.0</kp>
-			<kd>1.0</kd>
+			<mu1>1.0</mu1>
+			<mu2>1.0</mu2>
+			<kp>500000.0</kp>
+			<kd>1000.0</kd>
+			<minDepth>0.00</minDepth>
+			<maxVel>0.00</maxVel>
 		</gazebo>
 		<gazebo reference="${name}_little_proximal_link">
@@ -466,8 +500,10 @@
 			<!--selfCollide>true</selfCollide-->
 			<gravity>true</gravity>
-			<mu1>500.0</mu1>
-			<mu2>500.0</mu2>
-			<kp>10000000.0</kp>
-			<kd>1.0</kd>
+			<mu1>1.0</mu1>
+			<mu2>1.0</mu2>
+			<kp>500000.0</kp>
+			<kd>1000.0</kd>
+			<minDepth>0.00</minDepth>
+			<maxVel>0.00</maxVel>
 		</gazebo>
 		<gazebo reference="${name}_little_middle_link">
@@ -490,8 +526,10 @@
 			<!--selfCollide>true</selfCollide-->
 			<gravity>true</gravity>
-			<mu1>500.0</mu1>
-			<mu2>500.0</mu2>
-			<kp>10000000.0</kp>
-			<kd>1.0</kd>
+			<mu1>1.0</mu1>
+			<mu2>1.0</mu2>
+			<kp>500000.0</kp>
+			<kd>1000.0</kd>
+			<minDepth>0.00</minDepth>
+			<maxVel>0.00</maxVel>
 		</gazebo>
 		<gazebo reference="${name}_little_distal_link">
@@ -514,8 +552,10 @@
 			<!-- selfCollide>true</selfCollide-->
 			<gravity>true</gravity>
-			<mu1>500.0</mu1>
-			<mu2>500.0</mu2>
-			<kp>10000000.0</kp>
-			<kd>1.0</kd>
+			<mu1>1.0</mu1>
+			<mu2>1.0</mu2>
+			<kp>500000.0</kp>
+			<kd>1000.0</kd>
+			<minDepth>0.00</minDepth>
+			<maxVel>0.00</maxVel>
 		</gazebo>
 		<!-- JOINTS -->
@@ -620,4 +660,31 @@
 			<xacro:insert_block name="gazebo_joint_elements"/>
 		</gazebo>
+<!-- 		<gazebo>
+                     <plugin name="${name}_gazebo_gripper" filename="libvito_gazebo_gripper.so">
+		    <updateRate>1000.0</updateRate>
+		       <gripperAttachLink>${name}_thumb_knuckle_link</gripperAttachLink>
+ 		       <gripperLink>${name}_thumb_distal_link</gripperLink>
+		       <gripperLink>${name}_thumb_proximal_link</gripperLink>
+		        <gripperLink>${name}_index_knuckle_link</gripperLink>
+			<gripperLink>${name}_index_proximal_link</gripperLink>
+			<gripperLink>${name}_index_middle_link</gripperLink>
+ 			<gripperLink>${name}_index_distal_link</gripperLink>
+			<gripperLink>${name}_middle_knuckle_link</gripperLink>
+			<gripperLink>${name}_middle_proximal_link</gripperLink>
+                       <gripperLink>${name}_middle_middle_link</gripperLink>
+ 			<gripperLink>${name}_middle_distal_link</gripperLink>
+			<gripperLink>${name}_ring_knuckle_link</gripperLink>
+			<gripperLink>${name}_ring_proximal_link</gripperLink>
+			<gripperLink>${name}_ring_middle_link</gripperLink>
+                        <gripperLink>${name}_ring_distal_link</gripperLink>
+			<gripperLink>${name}_little_knuckle_link</gripperLink>
+			<gripperLink>${name}_little_proximal_link</gripperLink>
+                       <gripperLink>${name}_little_middle_link</gripperLink>
+ 			<gripperLink>${name}_little_distal_link</gripperLink>
+                       <maxRelativeMotionRate>0.001</maxRelativeMotionRate>
+                       <attachWait>0.1</attachWait>
+                       <detachWait>0.0</detachWait>
+                   </plugin>
+		 </gazebo>   -->
 	</xacro:macro>
 </robot>

File: soft_hand_description/model/soft_hand.inertia.xacro (robot description, xacro)
@@ -9,6 +9,6 @@
     <!-- I couldn't make the simulation work with realistic values, so I tweaked the conversion values -->
     <xacro:property name="mm_to_m" value="0.001"/>
-    <xacro:property name="mm2_to_m2" value="0.001"/>
-    <xacro:property name="gr_to_Kg" value="0.01"/>
+   <xacro:property name="mm2_to_m2" value="0.001"/>
+    <xacro:property name="gr_to_Kg" value="0.01"/>-
     <!-- not so negligible, otherwise simulation fails -->
     <xacro:property name="negligible_mass" value="${10*gr_to_Kg}"/>

File: soft_hand_description/model/soft_hand.transmission.xacro (robot description, xacro)
@@ -149,6 +149,6 @@
             <role>joint1</role>
             <offset>-0.0</offset>
-            <mechanicalReduction>1.3</mechanicalReduction>
-            <mechanicalElasticity>1.0</mechanicalElasticity>
+            <mechanicalReduction>0.6</mechanicalReduction>
+            <mechanicalElasticity>0.6</mechanicalElasticity>
             <!-- hardwareInterface>PositionJointInterface</hardwareInterface -->
             <hardwareInterface>EffortJointInterface</hardwareInterface>
